File: VT220_keyboard.kicad_pcb (KiCad board)
At the start: 2 copper layers, 484.4 x 135.6 mm, 93 parts, among them J1 Conn_01x10_Pin, J10 SW_MX_2, J11 SW_MX_3, J12 SW_MX_2, J13 SW_MX_3, J14 SW_MX_4, J15 SW_MX_1, J16 SW_MX_1, J17 SW_MX_4, J18 SW_MX_3, J19 SW_MX_3, J2 Conn_01x10_Pin, J20 SW_MX_3, J21 SW_MX_3, J22 SW_MX_3_LONG, J23 SW_MX_3_LONG, J24 SW_MX_3, J25 SW_MX_3, J26 SW_MX_3, J27 SW_MX_2, J28 SW_MX_3_LONG, J29 SW_MX_3, J3 Conn_01x10_Pin, J30 SW_MX_3, J31 SW_MX_3, J32 SW_MX_2, J33 SW_MX_1, J34 SW_MX_1, J35 SW_MX_3, J36 SW_MX_3, J37 SW_MX_3, J38 SW_MX_1, J39 SW_MX_1, J40 SW_MX_1, J41 SW_MX_1, J42 SW_MX_1, J43 SW_MX_3, J44 SW_MX_3, J45 SW_MX_1, J46 SW_MX_3, J47 SW_MX_4, J48 SW_MX_4, J49 SW_MX_4, J50 SW_MX_3, J51 SW_MX_1, J52 SW_MX_1, J53 SW_MX_1, J54 Conn_01x10_Pin, J55 Conn_01x10_Pin, J56 Conn_01x10_Pin, J57 Conn_01x10_Pin, J58 Conn_01x10_Pin, J59 Conn_01x10_Pin, J60 Conn_01x10_Pin, J61 Conn_01x10_Pin, J62 Conn_01x01_Pin, J63 Conn_01x01_Pin, J64 Conn_01x01_Pin, J65 Conn_01x01_Pin, J66 Conn_01x01_Pin, J67 Conn_01x01_Pin, J68 Conn_01x01_Pin, J69 Conn_01x01_Pin, M1 STAB_MX_2u, M2 STAB_MX_2u, M3 STAB_MX_2u, M4 STAB_MX_7u, M5 STAB_MX_6.25u, M6 STAB_MX_2u, M7 STAB_MX_2u, M8 STAB_MX_2u

Commit message: Update PCB
Routing:
- net 25: track 910.3 -> 897.0 mm
- net 4: track 540.4 -> 549.6 mm
- net 26: track 863.6 -> 869.8 mm
- net 23: track 871.4 -> 876.8 mm
- net 17: track 626.4 -> 630.8 mm
- net 14: track 196.9 -> 201.3 mm
- net 7: track 420.1 -> 424.3 mm
- net 16: track 498.9 -> 495.6 mm, vias 6 -> 5
- net 10: track 270.7 -> 267.8 mm
- net 13: track 916.0 -> 913.4 mm
- net 8: track 334.7 -> 337.1 mm
- net 20: track 514.2 -> 515.6 mm
- net 19: track 552.3 -> 553.6 mm
- net 18: track 850.2 -> 851.4 mm
- net 1: track 501.5 -> 502.5 mm
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Other:
- outline, holes or cut-outs redrawn
